File: fl_2k_vhf_uhf_Diplexer_10W.sch (KiCad schematic (older format))
At the start: 70 parts, among them J1 3mm mount, J2 3mm mount, J3 3mm mount, J4 3mm mount

Commit message: aded missing componenets
Parts:
- added C? (x5): C, symbol C
- added L?: L, symbol L
- added R?: R, symbol R
Connections:
- net +5V: now also U?.10 (Power_Down), U?.2 (V_BIAS), C?.1, C?.1, C?.1, R?.2
- net GND: now also C?.2, C?.2, C?.2, C?.2, C?.2
- net at J?.1 (Pin_1), J?.2 (Pin_2): now also C?.1, L?.2; no longer U?.3 (RF_in)
- net at U?.1 (V_BA1): now also R?.1
- new net: L?.1, U?.3 (RF_in)
Other:
- note added: "3.5V =1.5W"
- note added: "TO DO\n1) Power Down"
Changed lines of the file:
@@
 	2800 3600 3050 3600
-Wire Wire Line
-	3050 5450 3650 5450
 Wire Wire Line
 	5050 2400 5050 2700
@@
 Wire Wire Line
 	6350 4950 6350 5400
-Wire Wire Line
-	3050 3600 3050 5450
 $Comp
 L R R?
@@
 Wire Wire Line
 	4800 1550 4800 1650
+$Comp
+L R R?
+U 1 1 5B0885BE
+P 3500 5000
+F 0 "R?" V 3580 5000 50  0000 C CNN
+F 1 "R" V 3500 5000 50  0000 C CNN
+F 2 "" V 3430 5000 50  0001 C CNN
+F 3 "" H 3500 5000 50  0001 C CNN
+	1    3500 5000
+	-1   0    0    1
+$EndComp
+$Comp
+L C C?
+U 1 1 5B0885C4
+P 3150 5000
+F 0 "C?" H 3175 5100 50  0000 L CNN
+F 1 "C" H 3175 4900 50  0000 L CNN
+F 2 "" H 3188 4850 50  0001 C CNN
+F 3 "" H 3150 5000 50  0001 C CNN
+	1    3150 5000
+	1    0    0    -1
+$EndComp
+$Comp
+L +5V #PWR?
+U 1 1 5B0885CA
+P 3450 3950
+F 0 "#PWR?" H 3450 3800 50  0001 C CNN
+F 1 "+5V" H 3450 4090 50  0000 C CNN
+F 2 "" H 3450 3950 50  0001 C CNN
+F 3 "" H 3450 3950 50  0001 C CNN
+	1    3450 3950
+	1    0    0    -1
+$EndComp
+$Comp
+L C C?
+U 1 1 5B0885D0
+P 3150 4100
+F 0 "C?" H 3175 4200 50  0000 L CNN
+F 1 "C" H 3175 4000 50  0000 L CNN
+F 2 "" H 3188 3950 50  0001 C CNN
+F 3 "" H 3150 4100 50  0001 C CNN
+	1    3150 4100
+	1    0    0    -1
+$EndComp
+$Comp
+L GND #PWR?
+U 1 1 5B0885D6
+P 3150 4350
+F 0 "#PWR?" H 3150 4100 50  0001 C CNN
+F 1 "GND" H 3150 4200 50  0000 C CNN
+F 2 "" H 3150 4350 50  0001 C CNN
+F 3 "" H 3150 4350 50  0001 C CNN
+	1    3150 4350
+	1    0    0    -1
+$EndComp
+Wire Wire Line
+	3150 3950 3450 3950
+Wire Wire Line
+	3150 4850 3500 4850
+Connection ~ 3350 4850
+Connection ~ 3350 3950
+Wire Wire Line
+	3150 4250 3150 4350
+$Comp
+L GND #PWR?
+U 1 1 5B08888F
+P 3150 5150
+F 0 "#PWR?" H 3150 4900 50  0001 C CNN
+F 1 "GND" H 3150 5000 50  0000 C CNN
+F 2 "" H 3150 5150 50  0001 C CNN
+F 3 "" H 3150 5150 50  0001 C CNN
+	1    3150 5150
+	1    0    0    -1
+$EndComp
+Wire Wire Line
+	3350 3950 3350 5300
+Wire Wire Line
+	3350 5300 3650 5300
+Wire Wire Line
+	3650 5150 3500 5150
+Text Notes 5550 3650 0    60   ~ 0
+TO DO\n1) Power Down
+Text Notes 4450 800  0    60   ~ 0
+TO DO\n1) Power Down
+$Comp
+L +5V #PWR?
+U 1 1 5B08A875
+P 4550 4350
+F 0 "#PWR?" H 4550 4200 50  0001 C CNN
+F 1 "+5V" H 4550 4490 50  0000 C CNN
+F 2 "" H 4550 4350 50  0001 C CNN
+F 3 "" H 4550 4350 50  0001 C CNN
+	1    4550 4350
+	1    0    0    -1
+$EndComp
+$Comp
+L C C?
+U 1 1 5B08AD59
+P 5050 4500
+F 0 "C?" H 5075 4600 50  0000 L CNN
+F 1 "C" H 5075 4400 50  0000 L CNN
+F 2 "" H 5088 4350 50  0001 C CNN
+F 3 "" H 5050 4500 50  0001 C CNN
+	1    5050 4500
+	1    0    0    -1
+$EndComp
+Wire Wire Line
+	4550 4350 5050 4350
+Wire Wire Line
+	4550 4550 4550 4350
+$Comp
+L GND #PWR?
+U 1 1 5B08B052
+P 5050 4700
+F 0 "#PWR?" H 5050 4450 50  0001 C CNN
+F 1 "GND" H 5050 4550 50  0000 C CNN
+F 2 "" H 5050 4700 50  0001 C CNN
+F 3 "" H 5050 4700 50  0001 C CNN
+	1    5050 4700
+	1    0    0    -1
+$EndComp
+Wire Wire Line
+	5050 4650 5050 4700
+Text Notes 4600 3450 0    60   ~ 0
+3.5V =1.5W
+Text Notes 4700 6250 0    60   ~ 0
+3.5V =1.5W
+$Comp
+L L L?
+U 1 1 5B08C215
+P 3150 5450
+F 0 "L?" V 3100 5450 50  0000 C CNN
+F 1 "L" V 3225 5450 50  0000 C CNN
+F 2 "" H 3150 5450 50  0001 C CNN
+F 3 "" H 3150 5450 50  0001 C CNN
+	1    3150 5450
+	0    1    1    0
+$EndComp
+$Comp
+L C C?
+U 1 1 5B08C21B
+P 3400 5600
+F 0 "C?" H 3425 5700 50  0000 L CNN
+F 1 "C" H 3425 5500 50  0000 L CNN
+F 2 "" H 3438 5450 50  0001 C CNN
+F 3 "" H 3400 5600 50  0001 C CNN
+	1    3400 5600
+	1    0    0    -1
+$EndComp
+$Comp
+L C C?
+U 1 1 5B08C221
+P 2900 5600
+F 0 "C?" H 2925 5700 50  0000 L CNN
+F 1 "C" H 2925 5500 50  0000 L CNN
+F 2 "" H 2938 5450 50  0001 C CNN
+F 3 "" H 2900 5600 50  0001 C CNN
+	1    2900 5600
+	1    0    0    -1
+$EndComp
+$Comp
+L GND #PWR?
+U 1 1 5B08C227
+P 3400 5850
+F 0 "#PWR?" H 3400 5600 50  0001 C CNN
+F 1 "GND" H 3400 5700 50  0000 C CNN
+F 2 "" H 3400 5850 50  0001 C CNN
+F 3 "" H 3400 5850 50  0001 C CNN
+	1    3400 5850
+	1    0    0    -1
+$EndComp
+$Comp
+L GND #PWR?
+U 1 1 5B08C22D
+P 2900 5850
+F 0 "#PWR?" H 2900 5600 50  0001 C CNN
+F 1 "GND" H 2900 5700 50  0000 C CNN
+F 2 "" H 2900 5850 50  0001 C CNN
+F 3 "" H 2900 5850 50  0001 C CNN
+	1    2900 5850
+	1    0    0    -1
+$EndComp
+Wire Wire Line
+	2900 5750 2900 5850
+Wire Wire Line
+	3400 5750 3400 5850
+Wire Wire Line
+	3650 5450 3300 5450
+Wire Wire Line
+	3050 3600 3050 4850
+Wire Wire Line
+	3050 4850 2900 4850
+Wire Wire Line
+	2900 4850 2900 5450
+Wire Wire Line
+	2900 5450 3000 5450
 $EndSCHEMATC

Commit message: added anotation to Diagram
Parts:
- added C1: 47uF 16V Elec, symbol CP
- added C17, C29: 100pF, symbol C
- added C2, C4: 1nF, symbol C
- added C26: 18pF, symbol C
- added C3: 47uF 16V, symbol CP
- added D1: RL207, symbol D
- added J1: 3sip200, RPi_Hat:Samtec_HLE-120-02-XXX-DV-BE-XX-XX, symbol Conn_01x03
- added R10, R12, R15, R9: 0, Resistors_SMD:R_0805_HandSoldering, symbol R
- added R11, R16: OC, Resistors_SMD:R_0805_HandSoldering, symbol R
- C10: renamed from C?; value C -> 1000pF
- C11, C15, C16, C23, C24, C8: renamed from C?; value C -> 100pF
- C12, C25: renamed from C?; value C -> 220pF
- C13: renamed from C?; value C -> 15pF
- C14: renamed from C?; value C -> 27pF
- C18, C20, C5, C6: renamed from C?; value C -> 1uF 16V
- C19: renamed from C?; value C -> 2.4pF
- C21: renamed from C?; value C -> 1nF
- C22, C9: renamed from C?; value C -> 4.7uF 16V
- C27, C28: renamed from C?; value C -> n/c
- C30: renamed from C?; value C -> 10nF
- C7: renamed from C?; value C -> 3.3pF
- D2, D3, D4: renamed from D?; footprint (none) -> LEDs:LED_0805_HandSoldering
- F1: renamed from F?; footprint (none) -> Bacar:LFCN-80
- J2: renamed from J1; footprint Mounting_Holes:MountingHole_3.2mm_M3_Pad -> RPi_Hat:Pin_Header_Straight_2x20
- L1, L2, L3, L5: renamed from L?; value L -> 33nH
- L10, L4: renamed from L?; value L -> 22nH
- L6, L8: renamed from L?; value L -> 5.6nH
- L7: renamed from L?; value L -> 12nH
- L9: renamed from L?; value L -> 3.9nH
- R1, R22: renamed from R?; value R -> 1k8; footprint (none) -> Resistors_SMD:R_0805_HandSoldering
- R13: renamed from R?; value R -> 330; footprint (none) -> Resistors_SMD:R_0805_HandSoldering
- R14, R25: renamed from R?; value OC -> 220; footprint (none) -> Resistors_SMD:R_0805_HandSoldering
- R17: renamed from R?; value R -> 2k0; footprint (none) -> Resistors_SMD:R_0805_HandSoldering
- R18, R19, R20, R21, R23, R24, R3, R4, R5, R6, R7, R8: renamed from R?; footprint (none) -> Resistors_SMD:R_0805_HandSoldering
- R2: renamed from R?; value R -> 2k2; footprint (none) -> Resistors_SMD:R_0805_HandSoldering
- U2, U4: renamed from U?; footprint (none) -> Housings_DFN_QFN:QFN-12-1EP_3x3mm_Pitch0.5mm
- gave numbers to parts that had none: 15
- renumbered J2 to J3, J3 to J4, J4 to J5
Connections:
- net +5V: now also C10.1, C22.1, C3.1, C4.1, J1.2 (Pin_2)
- net GND: now also C1.2, C17.2, C2.2, C26.1, C29.2, C3.2, C4.2, J1.1 (Pin_1), R11.1, R16.1
- net at J6.1 (Pin_1), J8.1 (Pin_1): now also R10.1; no longer C15.2
- net at J6.2 (Pin_2), L4.2: now also C13.1
- net at J9.2 (Pin_2): now also R15.1; no longer C16.1
- net at L1.2, U2.11 (Vcc1): now also C7.1
- net at L4.1, U2.3 (RF_in): now also C14.1
- net at L6.2, U4.11 (Vcc1): now also C19.1
- net at L9.1, U4.3 (RF_in): now also C28.1
- net at L8.1, R18.2: now also C26.2
- net at U1.1 (VI): now also C1.1, C2.1, D1.1 (K)
- net at C12.1, L3.2: now also L5.1
- net at C25.1, L8.2: now also L10.1
- net at D3.2 (A), R14.1: now also C17.1
- net at D4.2 (A), R25.1: now also C29.1
- new net: C16.1, R12.2
- new net: C15.2, R9.2
- new net: R10.2, R11.2, R9.1
- new net: D1.2 (A), J1.3 (Pin_3)
- new net: R12.1, R15.2, R16.2
- no-connect marks 4 -> 10
Other:
- note added: "2m"
- note added: "UHF 70cm"
- note added: "VHF 2M"
- note removed: "40M"
- note removed: "40m Low Pass"
- note removed: "TO DO\n1) Power Down"
- note removed: "To Do:\nadd rf amps +27dbm\n\nMMZ09332BT1"
- moved on the sheet: C15, C16, C28, F1, J8, P1, R17, R5, R6, R8
